Commit message: Create wall.xacro
remove some comments to make it readable and clear

File: wall.xacro (robot description, xacro)
@@ -4,13 +4,4 @@
   <xacro:property name="length" value="1" />
   <xacro:property name="height" value="1" />
-  <!--<xacro:macro name="inertial_matrix" params="mass">
-      <inertial>
-      	<mass value="${mass}" />-->
-        <!-- below inertia tag has something wrong, because I confuse xacro:property with xacro:macro params-->
-        <!--<inertia ixx="${1.0/12*mass*(height**2+length**2)}" ixy="0.0" ixz="0.0" iyy="${1.0/12*mass*(width**2+length**2)}" iyz="0.0" izz="${1.0/12*mass*(height**2+width**2)}" />-->
-      <!--<inertia ixx="166.6666667" ixy="0.0" ixz="0.0" iyy="166.6666667" iyz="0.0" izz="166.6666667" />
-      </inertial>
-   </xacro:macro>-->
-<!--The inertia version without origin -->
  <xacro:macro name="box_inertial" params="x y z mass">
     <inertial>
@@ -21,14 +12,4 @@
     </inertial>
   </xacro:macro>
-  <!--The inertia version with origin -->
-   <!--<xacro:macro name="box_inertial_with_origin" params="x y z mass *origin">
-    <inertial>
-      <mass value="${mass}" />
-      <insert_block name="origin"/>
-      <inertia ixx="${0.0833333 * mass * (y*y + z*z)}" ixy="0.0" ixz="0.0"
-        iyy="${0.0833333 * mass * (x*x + z*z)}" iyz="0.0"
-        izz="${0.0833333 * mass * (x*x + y*y)}" />
-    </inertial>
-  </xacro:macro>-->
   <link name="wall_link">
       <visual>
@@ -46,8 +27,4 @@
       </collision>
 <xacro:box_inertial mass="1000" x="1" y="1" z="1"/>
-<!--<xacro:box_inertial_with_origin mass="1000" x="1" y="1" z="1">
-  <origin xyz="0 0 ${-height/2.0}" rpy="0 0 0"/>
-</xacro:box_inertial_with_origin>-->
-      <!--<xacro:inertial_matrix mass="1000"/>-->
     </link>
     <gazebo reference="wall_link">
